File: USBDroidR3.brd (EAGLE design)
At the start: 68.6 x 53.3 mm, 90 parts, among them IC1 LD29150DT50R, IC2 ATMEGA16U2-MU, IC3 LM358D, IC4 MAX3421EEHJ, IC5 ATMEGA328P TQFP32, IC6 74HC4050 SOIC16, J1 DC_2_1MM, P1 USBSF-MICROB, P2 ICSP:MAIN, P3 USB_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

Commit message: R3 updates
Parts:
- P1: value USBSF-MICROB -> USB-6PSMT; device freetronics-jon:USB-MICROB -> freetronics-jon:USB-MICROB-MB05PMXX
- moved SJ1 2.05 mm to (5.19, 43.7)
Connections:
- net N$51: now also P1.PIN1, P1.PIN2
Routing:
- net N$51: track 35.3 -> 40.0 mm, vias 0 -> 2
- net N$47: track 20.2 -> 18.2 mm
Other:
- board text added: "Analog Inputs"
- board text added: "I2C"
- board text added: "R3"
- board text added: "v2.0"
- board text removed: "Analog"
- board text removed: "v1.1"

Commit message: Updated designators, ERC and DRC for release
Parts:
- H1: value M100.1 -> Digital_8_13
- H2: value (none) -> Power
- moved D1 8.77 mm to (24.8, 9.65), turned to 180 degrees
- moved C4 6.55 mm to (22.4, 4.06), turned to 180 degrees
- moved C3 5.49 mm to (17.5, 9.65), turned to 270 degrees
- moved C15 3.81 mm to (27.4, 13.0), turned to 180 degrees
- moved C16 3.05 mm to (23.1, 13.0)
- renumbered JP2 to H2, JP3 to H1
Connections:
- net N$47 renamed USBGND
Routing:
- net VIN: track 104.5 -> 120.2 mm
- net N$60: track 4.24 -> 11.4 mm
- net 5V: track 292.0 -> 295.8 mm
- net N$30: track 11.9 -> 14.1 mm
- net N$27: track 8.55 -> 10.4 mm
- net N$51: track 40.0 -> 39.1 mm
- net N$115: track 13.4 -> 12.7 mm
Other:
- board text added: "Analog"
- board text removed: "Analog Inputs"
