File: USBDroidR3.sch (EAGLE design)
At the start: 90 parts, among them IC1 LD29150DT50R, IC2 ATMEGA16U2-MU, IC3 LM358D, IC4 MAX3421EEHJ, IC5 ATMEGA328P TQFP32, IC6 74HC4050 SOIC16, J1 DC_2_1MM, P1 USBSF-MICROB, P2 ICSP:MAIN, P3 USB_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

Commit message: R3 updates
Parts:
- P1: value USBSF-MICROB -> USB-6PSMT; device freetronics-jon:USBSF-MICROB -> freetronics-jon:USB-6PSMT
Connections:
- net N$51: now also P1.PIN1, P1.PIN2
Other:
- note added: "Freetronics USBDroid R3"
- note added: "V2.0 (2012-07-06)"
- note added: "www.freetronics.com/usbdroid"
Changed lines of the file:
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@@
 <part name="L2" library="freetronics-master-v1" deviceset="INDUCTOR" device="0805-LARGE" value="0805 INDUCTOR"/>
 <part name="C9" library="freetronics" deviceset="CAP" device="0603" value="1uF 0603"/>
-<part name="P1" library="freetronics-jon" deviceset="USBSF" device="-MICROB"/>
+<part name="P1" library="freetronics-jon" deviceset="USB-6P" device="SMT"/>
 <part name="GND38" library="SparkFun" deviceset="GND" device=""/>
 <part name="GND39" library="SparkFun" deviceset="GND" device=""/>
@@
 <text x="261.62" y="96.52" size="1.778" layer="94">In Circuit Serial Programming</text>
 <text x="261.62" y="48.26" size="1.778" layer="94">micro SD Card Slot</text>
-<text x="396.24" y="12.7" size="2.794" layer="94">Freetronics USBDroid (Arduino Compatible)</text>
-<text x="469.9" y="6.858" size="1.778" layer="94">V1.1 (2011-06-01)</text>
-<text x="436.626" y="6.858" size="1.778" layer="94">www.freetronics.com</text>
+<text x="396.24" y="12.7" size="2.794" layer="94">Freetronics USBDroid R3</text>
+<text x="469.9" y="6.858" size="1.778" layer="94">V2.0 (2012-07-06)</text>
+<text x="421.386" y="6.858" size="1.778" layer="94">www.freetronics.com/usbdroid</text>
 <text x="396.24" y="6.858" size="1.778" layer="94">SKU: USBDROID</text>
 <text x="241.3" y="271.78" size="1.6764" layer="94" ratio="12" rot="R90">D4 used by microSD card Chip Select.</text>
@@
 <frame x1="254" y1="0" x2="502.92" y2="185.42" columns="8" rows="5" layer="94"/>
 <frame x1="393.7" y1="5.08" x2="497.84" y2="17.78" columns="0" rows="0" layer="94" border-left="no" border-top="no" border-right="no" border-bottom="no"/>
-<frame x1="393.7" y1="5.08" x2="431.8" y2="10.16" columns="8" rows="5" layer="94"/>
+<frame x1="393.7" y1="5.08" x2="419.1" y2="10.16" columns="8" rows="5" layer="94"/>
 <frame x1="467.36" y1="5.08" x2="497.84" y2="10.16" columns="8" rows="5" layer="94"/>
 <wire x1="355.6" y1="145.796" x2="355.6" y2="100.33" width="0.4064" layer="97" style="longdash"/>
@@
 <attribute name="VALUE" x="403.098" y="140.335" size="1.778" layer="96"/>
 </instance>
-<instance part="P1" gate="G$1" x="386.08" y="127" rot="R180"/>
+<instance part="P1" gate="G$1" x="381" y="127" rot="R180"/>
 <instance part="GND38" gate="1" x="429.26" y="132.08"/>
 <instance part="GND39" gate="1" x="431.8" y="101.6" smashed="yes">
@@
 <segment>
 <wire x1="396.24" y1="119.38" x2="396.24" y2="127" width="0.1524" layer="91"/>
-<wire x1="396.24" y1="127" x2="391.16" y2="127" width="0.1524" layer="91"/>
+<wire x1="396.24" y1="127" x2="386.08" y2="127" width="0.1524" layer="91"/>
 <wire x1="396.24" y1="127" x2="406.4" y2="127" width="0.1524" layer="91"/>
 <wire x1="406.4" y1="127" x2="406.4" y2="119.38" width="0.1524" layer="91"/>
@@
 <segment>
 <wire x1="398.78" y1="119.38" x2="398.78" y2="129.54" width="0.1524" layer="91"/>
-<wire x1="398.78" y1="129.54" x2="391.16" y2="129.54" width="0.1524" layer="91"/>
+<wire x1="398.78" y1="129.54" x2="386.08" y2="129.54" width="0.1524" layer="91"/>
 <wire x1="414.02" y1="121.92" x2="408.94" y2="121.92" width="0.1524" layer="91"/>
 <wire x1="408.94" y1="121.92" x2="408.94" y2="129.54" width="0.1524" layer="91"/>
@@
 <net name="N$115" class="0">
 <segment>
-<wire x1="396.24" y1="132.08" x2="391.16" y2="132.08" width="0.1524" layer="91"/>
+<wire x1="396.24" y1="132.08" x2="386.08" y2="132.08" width="0.1524" layer="91"/>
 <pinref part="F1" gate="G$1" pin="1"/>
 <pinref part="P1" gate="G$1" pin="VBUS"/>
@@
 <wire x1="416.56" y1="104.14" x2="416.56" y2="109.22" width="0.1524" layer="91"/>
 <wire x1="416.56" y1="109.22" x2="419.1" y2="109.22" width="0.1524" layer="91"/>
-<wire x1="391.16" y1="121.92" x2="403.86" y2="121.92" width="0.1524" layer="91"/>
+<wire x1="386.08" y1="121.92" x2="403.86" y2="121.92" width="0.1524" layer="91"/>
 <wire x1="403.86" y1="121.92" x2="403.86" y2="109.22" width="0.1524" layer="91"/>
 <wire x1="403.86" y1="109.22" x2="416.56" y2="109.22" width="0.1524" layer="91"/>
@@
 <segment>
 <pinref part="P1" gate="G$1" pin="TAB1"/>
-<wire x1="386.08" y1="137.16" x2="386.08" y2="142.24" width="0.1524" layer="91"/>
-<wire x1="386.08" y1="142.24" x2="383.54" y2="142.24" width="0.1524" layer="91"/>
+<wire x1="381" y1="139.7" x2="381" y2="142.24" width="0.1524" layer="91"/>
+<wire x1="381" y1="142.24" x2="378.46" y2="142.24" width="0.1524" layer="91"/>
 <pinref part="P1" gate="G$1" pin="FIX1"/>
-<wire x1="383.54" y1="142.24" x2="383.54" y2="137.16" width="0.1524" layer="91"/>
-<wire x1="383.54" y1="142.24" x2="378.46" y2="142.24" width="0.1524" layer="91"/>
-<wire x1="378.46" y1="142.24" x2="378.46" y2="104.14" width="0.1524" layer="91"/>
-<wire x1="383.54" y1="104.14" x2="386.08" y2="104.14" width="0.1524" layer="91"/>
-<wire x1="386.08" y1="104.14" x2="396.24" y2="104.14" width="0.1524" layer="91"/>
+<wire x1="378.46" y1="142.24" x2="378.46" y2="139.7" width="0.1524" layer="91"/>
+<wire x1="378.46" y1="142.24" x2="368.3" y2="142.24" width="0.1524" layer="91"/>
+<wire x1="368.3" y1="142.24" x2="368.3" y2="104.14" width="0.1524" layer="91"/>
+<wire x1="378.46" y1="104.14" x2="381" y2="104.14" width="0.1524" layer="91"/>
+<wire x1="381" y1="104.14" x2="388.62" y2="104.14" width="0.1524" layer="91"/>
+<wire x1="388.62" y1="104.14" x2="396.24" y2="104.14" width="0.1524" layer="91"/>
 <wire x1="396.24" y1="104.14" x2="398.78" y2="104.14" width="0.1524" layer="91"/>
 <wire x1="396.24" y1="109.22" x2="396.24" y2="104.14" width="0.1524" layer="91"/>
@@
 <pinref part="L2" gate="G$1" pin="1"/>
 <pinref part="P1" gate="G$1" pin="FIX2"/>
-<wire x1="383.54" y1="104.14" x2="383.54" y2="116.84" width="0.1524" layer="91"/>
+<wire x1="378.46" y1="104.14" x2="378.46" y2="114.3" width="0.1524" layer="91"/>
 <pinref part="P1" gate="G$1" pin="TAB2"/>
-<wire x1="386.08" y1="116.84" x2="386.08" y2="104.14" width="0.1524" layer="91"/>
-<wire x1="378.46" y1="104.14" x2="383.54" y2="104.14" width="0.1524" layer="91"/>
-<junction x="383.54" y="142.24"/>
-<junction x="383.54" y="104.14"/>
-<junction x="386.08" y="104.14"/>
-</segment>
-</net>
+<wire x1="381" y1="114.3" x2="381" y2="104.14" width="0.1524" layer="91"/>
+<wire x1="368.3" y1="104.14" x2="378.46" y2="104.14" width="0.1524" layer="91"/>
+<junction x="378.46" y="142.24"/>
+<junction x="378.46" y="104.14"/>
+<junction x="381" y="104.14"/>
+<pinref part="P1" gate="G$1" pin="PIN1"/>
+<wire x1="386.08" y1="134.62" x2="388.62" y2="134.62" width="0.1524" layer="91"/>
+<wire x1="388.62" y1="134.62" x2="388.62" y2="142.24" width="0.1524" layer="91"/>
+<wire x1="388.62" y1="142.24" x2="381" y2="142.24" width="0.1524" layer="91"/>
+<pinref part="P1" gate="G$1" pin="PIN2"/>
+<wire x1="386.08" y1="119.38" x2="388.62" y2="119.38" width="0.1524" layer="91"/>
+<wire x1="388.62" y1="119.38" x2="388.62" y2="104.14" width="0.1524" layer="91"/>
+<junction x="381" y="142.24"/>
+<junction x="388.62" y="104.14"/>
+</segment>
+</net>

Commit message: Updated designators, ERC and DRC for release
Parts:
- H1: value M100.1 -> Digital_8_13
- H2: value (none) -> Power
- renumbered JP2 to H2, JP3 to H1
Connections:
- net N$47 renamed USBGND
Other:
- note added: "(Linked)"
- note added: "Short across SJ3 RESET-EN and SJ1 GROUND after all other routing is complete"
- note removed: "Freetronics USBDroid (Arduino Compatible)"
- note removed: "V1.1 (2011-06-01)"
- note removed: "www.freetronics.com"
- moved on the sheet: A1, A2, C14, C17, C18, C22, IC5, LED5, P1, Q2, R10, R3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
